Commit message: feat: Serial Chain, Reach Samples, TreeFK preview (Motus.NET 0.7.1)
Parametric Motus Serial Chain + capped Reach Samples; URDF tip visuals posed via Motus.NET TreeFK/mimic. Pin MotusNetPackages to 0.7.1. ADR 0002.

Co-authored-by: Cursor <cursoragent@cursor.com>

File: examples/ur10e/ur10e_robotiq.urdf (robot description, URDF)
Before this commit: robot ur10e_robotiq, 20 links, 19 joints
Joints:
- removed joint robotiq_base_left_inner
- removed joint robotiq_base_left_knuckle
- removed joint robotiq_base_right_inner
- removed joint robotiq_base_right_knuckle
- added joint robotiq_left_inner_knuckle: type revolute, parent robotiq_base, child robotiq_left_inner_knuckle, origin xyz=0.0127 0 0.06142 rpy=0 0 0, axis 0 -1 0, limit lower=0 upper=0.8 effort=50 velocity=0.5, mimic joint=robotiq_left_knuckle multiplier=1
- added joint robotiq_left_knuckle: type revolute, parent robotiq_base, child robotiq_left_knuckle, origin xyz=0.03060114 0 0.05490452 rpy=0 0 0, axis 0 -1 0, limit lower=0 upper=0.8 effort=50 velocity=0.5
- added joint robotiq_right_inner_knuckle: type revolute, parent robotiq_base, child robotiq_right_inner_knuckle, origin xyz=-0.0127 0 0.06142 rpy=0 0 0, axis 0 -1 0, limit lower=-0.8 upper=0 effort=50 velocity=0.5, mimic joint=robotiq_left_knuckle multiplier=-1
- added joint robotiq_right_knuckle: type revolute, parent robotiq_base, child robotiq_right_knuckle, origin xyz=-0.03060114 0 0.05490452 rpy=0 0 0, axis 0 -1 0, limit lower=-0.8 upper=0 effort=50 velocity=0.5, mimic joint=robotiq_left_knuckle multiplier=-1
- joint robotiq_left_finger_tip: axis (none) -> 0 -1 0; limit (none) -> lower=-0.8 upper=0 effort=50 velocity=0.5; mimic (none) -> joint=robotiq_left_knuckle multiplier=-1; type fixed -> revolute
- joint robotiq_right_finger_tip: axis (none) -> 0 -1 0; limit (none) -> lower=0 upper=0.8 effort=50 velocity=0.5; mimic (none) -> joint=robotiq_left_knuckle multiplier=1; type fixed -> revolute
