Commit message: fix(examples): readable 07 preview and overlap-safe layouts
ur10e_minimal had almost no visuals so Preview looked empty; add
primitive link meshes and rewrite 07 L→R. Widen Plan/Scrub/Preview
spacing for live chrome and regenerate all GHX.

Co-authored-by: Cursor <cursoragent@cursor.com>

File: examples/ur10e/ur10e_minimal.urdf (robot description, URDF)
Before this commit: robot ur10e_minimal, 7 links, 6 joints
Links:
- link base_link: geometry collision cylinder length=0.10 radius=0.08; visual cylinder length=0.10 radius=0.08
- link forearm_link: geometry collision box size=0.10 0.52 0.10; visual box size=0.10 0.52 0.10
- link shoulder_link: geometry collision cylinder length=0.14 radius=0.10; visual cylinder length=0.14 radius=0.10
- link tool0: geometry collision cylinder length=0.06 radius=0.04; visual cylinder length=0.06 radius=0.04
- link upper_arm_link: geometry collision box size=0.12 0.56 0.12; visual box size=0.12 0.56 0.12
- link wrist_1_link: geometry collision cylinder length=0.10 radius=0.05; visual cylinder length=0.10 radius=0.05
- link wrist_2_link: geometry collision cylinder length=0.10 radius=0.045; visual cylinder length=0.10 radius=0.045
